Commit message: Add standoffs and tray in barista robot

File: urdf/barista_robot_model.urdf (robot description, URDF)
Before this commit: robot barista_robot, 9 links, 8 joints
Links:
- added link standoff_1, mass 0.05; collision cylinder length=0.22 radius=0.01; visual cylinder length=0.22 radius=0.01
- added link standoff_2, mass 0.05; collision cylinder length=0.22 radius=0.01; visual cylinder length=0.22 radius=0.01
- added link standoff_3, mass 0.05; collision cylinder length=0.22 radius=0.01; visual cylinder length=0.22 radius=0.01
- added link standoff_4, mass 0.05; collision cylinder length=0.22 radius=0.01; visual cylinder length=0.22 radius=0.01
- added link tray, mass 0.3; collision cylinder length=0.09 radius=0.16; visual cylinder length=0.09 radius=0.16
Joints:
- added joint joint_standoff_1: type fixed, parent base_link, child standoff_1, origin xyz=0.1 0.1 0.0775
- added joint joint_standoff_2: type fixed, parent base_link, child standoff_2, origin xyz=0.1 -0.1 0.0775
- added joint joint_standoff_3: type fixed, parent base_link, child standoff_3, origin xyz=-0.1 -0.1 0.0775
- added joint joint_standoff_4: type fixed, parent base_link, child standoff_4, origin xyz=-0.1 0.1 0.0775
- added joint joint_tray: type fixed, parent base_link, child tray, origin xyz=0 0 0.2975

Commit message: Update cater and wheels position relative to base_link

File: urdf/barista_robot_model.urdf (robot description, URDF)
Before this commit: robot barista_robot, 14 links, 13 joints
Joints:
- joint back_yaw_joint: origin xyz=-0.15 0 -0.0775 rpy=0 0 0 -> xyz=-0.15 0 -0.0875 rpy=0 0 0
- joint front_yaw_joint: origin xyz=0.15 0 -0.0775 rpy=0 0 0 -> xyz=0.15 0 -0.0875 rpy=0 0 0
- joint joint_left_wheel: origin xyz=0 0.15 -0.0573 rpy=0 0 0 -> xyz=0 0.15 -0.0623 rpy=0 0 0
- joint joint_right_wheel: origin xyz=0 -0.15 -0.0573 rpy=0 0 0 -> xyz=0 -0.15 -0.0623 rpy=0 0 0

Commit message: Add laser scan functionality

File: urdf/barista_robot_model.urdf (robot description, URDF)
Before this commit: robot barista_robot, 14 links, 13 joints
Links:
- added link laser_scan_frame
- added link laser_scan_link, mass 0.01; collision cylinder length=0.0408 radius=0.037493; visual mesh filename=package://barista_robot_description/meshes/hokuyo_urg_04lx.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 scale=1.0 1.0 1.0
Joints:
- added joint laser_scan_frame_joint: type fixed, parent laser_scan_link, child laser_scan_frame, origin xyz=0.03 0 0.05 rpy=0 0 0
- added joint laser_scan_link_joint: type fixed, parent base_link, child laser_scan_link, origin xyz=0.12 0 0.0775 rpy=0 0 0

Commit message: Add colors to links

File: urdf/barista_robot_model.urdf (robot description, URDF)
Before this commit: robot barista_robot, 16 links, 15 joints
Links:
- link laser_scan_frame: mass None -> 1e-6

Commit message: Add base footprint link to barista urdf model

File: urdf/barista_robot_model.urdf (robot description, URDF)
Before this commit: robot barista_robot, 16 links, 15 joints
Links:
- added link base_footprint
Joints:
- added joint joint_base_link: type fixed, parent base_footprint, child base_link, origin xyz=0 0 0.0975 rpy=0 0 0

Commit message: Fix laser scan fram id and its position

File: urdf/barista_robot_model.urdf (robot description, URDF)
Before this commit: robot barista_robot, 17 links, 16 joints
Links:
- link laser_scan_link: mass 0.01 -> 0.015; geometry collision cylinder length=0.07 radius=0.025; visual mesh filename=package://barista_robot_description/meshes/hokuyo_urg_04lx.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 scale=1.0 1.0 1.0
Joints:
- joint laser_scan_frame_joint: origin xyz=0.03 0 0.05 rpy=0 0 0 -> xyz=0 0 0.06 rpy=0 0 0
- joint laser_scan_link_joint: origin xyz=0.12 0 0.0775 rpy=0 0 0 -> xyz=0.13 0 0.0775 rpy=0 0 0
