Commit message: Add caster and drive sheels xacro files

File: xacro/barista_robot_model.urdf.xacro (robot description, xacro)
@@ -1,4 +1,6 @@
 <?xml version="1.0"?>
 <robot xmlns:xacro="http://www.ros.org/wiki/xacro" name="barista_robot">
+  <xacro:include filename="$(find barista_robot_description)/xacro/drive_wheel.xacro" />
+  <xacro:include filename="$(find barista_robot_description)/xacro/caster_wheel.xacro" />
   <gazebo reference="base_link">
     <material>Gazebo/Blue</material>
@@ -97,231 +99,11 @@
   </link>
   <!-- Wheel Left -->
-  <link name="left_wheel">
-    <visual>
-      <origin rpy="0 1.5707 1.5707" xyz="0 0 0"/>
-      <geometry>
-        <cylinder length="0.0206" radius="0.0352"/>
-      </geometry>
-      <material name="black" />
-    </visual>
-    <collision>
-      <origin rpy="0 1.5707 1.5707" xyz="0 0 0"/>
-      <geometry>
-        <cylinder length="0.0206" radius="0.0352"/>
-      </geometry>
-    </collision>
-    <inertial>
-      <origin rpy="0 1.5707 1.5707" xyz="0 0 0"/>
-      <mass value="0.05"/>
-      <inertia ixx="0.00001725616667" ixy="0" ixz="0" iyy="0.00001725616667" iyz="0" izz="0.000030976"/>
-    </inertial>
-  </link>
-  <joint name="joint_left_wheel" type="continuous">
-    <origin rpy="0 0 0" xyz="0 0.15 -0.0623"/>
-    <child link="left_wheel"/>
-    <parent link="base_link"/>
-    <axis rpy="0 0 0" xyz="0 1 0"/>
-    <limit effort="10000" velocity="1000"/>
-    <joint_properties damping="1.0" friction="1.0"/>
-  </joint>
+  <xacro:wheel wheel_name="left_wheel" joint_origin="0 0.15 -0.0623"/>
   <!-- Wheel Right -->
-  <link name="right_wheel">
-    <visual>
-      <origin rpy="0 1.5707 1.5707" xyz="0 0 0"/>
-      <geometry>
-        <cylinder length="0.0206" radius="0.0352"/>
-      </geometry>
-      <material name="black" />
-    </visual>
-    <collision>
-      <origin rpy="0 1.5707 1.5707" xyz="0 0 0"/>
-      <geometry>
-        <cylinder length="0.0206" radius="0.0352"/>
-      </geometry>
-    </collision>
-    <inertial>
-      <origin rpy="0 1.5707 1.5707" xyz="0 0 0"/>
-      <mass value="0.05"/>
-      <inertia ixx="0.00001725616667" ixy="0" ixz="0" iyy="0.00001725616667" iyz="0" izz="0.000030976"/>
-    </inertial>
-  </link>
-  <joint name="joint_right_wheel" type="continuous">
-    <origin rpy="0 0 0" xyz="0 -0.15 -0.0623"/>
-    <child link="right_wheel"/>
-    <parent link="base_link"/>
-    <axis rpy="0 0 0" xyz="0 1 0"/>
-    <limit effort="10000" velocity="1000"/>
-    <joint_properties damping="1.0" friction="1.0"/>
-  </joint>
+  <xacro:wheel wheel_name="right_wheel" joint_origin="0 -0.15 -0.0623" />
   <!-- Caster Wheel Front -->
-  <link name="front_yaw_link">
-    <visual>
-      <origin rpy="0 1.5707 1.5707" xyz="0 0 0"/>
-      <geometry>
-        <cylinder length="0.001" radius="0.0045000000000000005"/>
-      </geometry>
-      <material name="blue" />
-    </visual>
-    <collision>
-      <origin rpy="0 1.5707 1.5707" xyz="0 0 0"/>
-      <geometry>
-        <cylinder length="0.001" radius="0.0045000000000000005"/>
-      </geometry>
-    </collision>
-    <inertial>
-        <origin rpy="0 1.5707 1.5707" xyz="0 0 0"/>
-        <mass value="0.001"/>
-        <inertia ixx="5.145833333333334e-09" ixy="0" ixz="0" iyy="5.145833333333334e-09" iyz="0" izz="1.0125000000000003e-08"/>
-    </inertial>
-  </link>
-  <joint name="front_yaw_joint" type="continuous">
-    <origin rpy="0 0 0" xyz="0.15 0 -0.0875" />
-    <parent link="base_link" />
-    <child link="front_yaw_link" />
-    <axis xyz="0 0 1" />
-    <limit effort="1000.0" velocity="100.0" />
-    <dynamics damping="0.0" friction="0.1"/>
-  </joint>
-  <link name="front_roll_link">
-    <visual>
-      <origin rpy="0 1.5707 1.5707" xyz="0 0 0"/>
-      <geometry>
-        <cylinder length="0.001" radius="0.0045000000000000005"/>
-      </geometry>
-      <material name="red" />
-    </visual>
-    <collision>
-      <origin rpy="0 1.5707 1.5707" xyz="0 0 0"/>
-      <geometry>
-        <cylinder length="0.001" radius="0.0045000000000000005"/>
-      </geometry>
-    </collision>
-    <inertial>
-        <origin rpy="0 1.5707 1.5707" xyz="0 0 0"/>
-        <mass value="0.001"/>
-        <inertia ixx="5.145833333333334e-09" ixy="0" ixz="0" iyy="5.145833333333334e-09" iyz="0" izz="1.0125000000000003e-08"/>
-    </inertial>
-  </link>
-  <joint name="front_roll_joint" type="continuous">
-    <origin rpy="0 0 0" xyz="0 0 0" />
-    <parent link="front_yaw_link" />
-    <child link="front_roll_link" />
-    <axis xyz="1 0 0" />
-    <limit effort="1000.0" velocity="100.0" />
-    <dynamics damping="0.0" friction="0.1"/>
-  </joint>
-  <link name="front_pitch_link">
-    <visual>
-      <origin rpy="0 1.5707 1.5707" xyz="0 0 0"/>
-      <geometry>
-        <sphere radius="0.010"/>
-      </geometry>
-      <material name="green" />
-    </visual>
-    <collision>
-      <origin rpy="0 1.5707 1.5707" xyz="0 0 0"/>
-      <geometry>
-        <sphere radius="0.010"/>
-      </geometry>
-    </collision>
-    <inertial>
-      <origin rpy="0 1.5707 1.5707" xyz="0 0 0"/>
-      <mass value="0.001"/>
-      <inertia ixx="4e-08" ixy="0" ixz="0" iyy="4e-08" iyz="0" izz="4e-08"/>
-    </inertial>
-  </link>
-  <joint name="front_pitch_joint" type="continuous">
-    <origin rpy="0 0 0" xyz="0 0 0" />
-    <parent link="front_roll_link" />
-    <child link="front_pitch_link" />
-    <axis xyz="0 1 0" />
-    <limit effort="1000.0" velocity="100.0" />
-    <dynamics damping="0.0" friction="0.1"/>
-  </joint>
-<!-- Caster Wheel Back -->
-  <link name="back_yaw_link">
-    <visual>
-      <origin rpy="0 1.5707 1.5707" xyz="0 0 0"/>
-      <geometry>
-        <cylinder length="0.001" radius="0.0045000000000000005"/>
-      </geometry>
-      <material name="blue" />
-    </visual>
-    <collision>
-      <origin rpy="0 1.5707 1.5707" xyz="0 0 0"/>
-      <geometry>
-        <cylinder length="0.001" radius="0.0045000000000000005"/>
-      </geometry>
-    </collision>
-    <inertial>
-        <origin rpy="0 1.5707 1.5707" xyz="0 0 0"/>
-        <mass value="0.001"/>
-        <inertia ixx="5.145833333333334e-09" ixy="0" ixz="0" iyy="5.145833333333334e-09" iyz="0" izz="1.0125000000000003e-08"/>
-    </inertial>
-  </link>
-  <joint name="back_yaw_joint" type="continuous">
-    <origin rpy="0 0 0" xyz="-0.15 0 -0.0875" />
-    <parent link="base_link" />
-    <child link="back_yaw_link" />
-    <axis xyz="0 0 1" />
-    <limit effort="1000.0" velocity="100.0" />
-    <dynamics damping="0.0" friction="0.1"/>
-  </joint>
-  <link name="back_roll_link">
-    <visual>
-      <origin rpy="0 1.5707 1.5707" xyz="0 0 0"/>
-      <geometry>
-        <cylinder length="0.001" radius="0.0045000000000000005"/>
-      </geometry>
-      <material name="red" />
-    </visual>
-    <collision>
-      <origin rpy="0 1.5707 1.5707" xyz="0 0 0"/>
-      <geometry>
-        <cylinder length="0.001" radius="0.0045000000000000005"/>
-      </geometry>
-    </collision>
-    <inertial>
-        <origin rpy="0 1.5707 1.5707" xyz="0 0 0"/>
-        <mass value="0.001"/>
-        <inertia ixx="5.145833333333334e-09" ixy="0" ixz="0" iyy="5.145833333333334e-09" iyz="0" izz="1.0125000000000003e-08"/>
-    </inertial>
-  </link>
-  <joint name="back_roll_joint" type="continuous">
-    <origin rpy="0 0 0" xyz="0 0 0" />
-    <parent link="back_yaw_link" />
-    <child link="back_roll_link" />
-    <axis xyz="1 0 0" />
-    <limit effort="1000.0" velocity="100.0" />
-    <dynamics damping="0.0" friction="0.1"/>
-  </joint>
-  <link name="back_pitch_link">
-    <visual>
-      <origin rpy="0 1.5707 1.5707" xyz="0 0 0"/>
-      <geometry>
-        <sphere radius="0.010"/>
-      </geometry>
-      <material name="green" />
-    </visual>
-    <collision>
-      <origin rpy="0 1.5707 1.5707" xyz="0 0 0"/>
-      <geometry>
-        <sphere radius="0.010"/>
-      </geometry>
-    </collision>
-    <inertial>
-        <origin rpy="0 1.5707 1.5707" xyz="0 0 0"/>
-        <mass value="0.001"/>
-        <inertia ixx="4e-08" ixy="0" ixz="0" iyy="4e-08" iyz="0" izz="4e-08"/>
-    </inertial>
-  </link>
-  <joint name="back_pitch_joint" type="continuous">
-    <origin rpy="0 0 0" xyz="0 0 0" />
-    <parent link="back_roll_link" />
-    <child link="back_pitch_link" />
-    <axis xyz="0 1 0" />
-    <limit effort="1000.0" velocity="100.0" />
-    <dynamics damping="0.0" friction="0.1"/>
-  </joint>
+  <xacro:caster caster_position="front" joint_yaw_origin="0.15 0 -0.0875" />
+  <!-- Caster Wheel Back -->
+  <xacro:caster caster_position="back" joint_yaw_origin="-0.15 0 -0.0875" />
    <!-- Standoff 1 -->
   <link name="standoff_1">

Commit message: Add standoff and tray xacro files

File: xacro/barista_robot_model.urdf.xacro (robot description, xacro)
@@ -3,4 +3,6 @@
   <xacro:include filename="$(find barista_robot_description)/xacro/drive_wheel.xacro" />
   <xacro:include filename="$(find barista_robot_description)/xacro/caster_wheel.xacro" />
+  <xacro:include filename="$(find barista_robot_description)/xacro/standoff_rod.xacro" />
+  <xacro:include filename="$(find barista_robot_description)/xacro/cup_holder_tray.xacro" />
   <gazebo reference="base_link">
     <material>Gazebo/Blue</material>
@@ -107,133 +109,13 @@
   <xacro:caster caster_position="back" joint_yaw_origin="-0.15 0 -0.0875" />
    <!-- Standoff 1 -->
-  <link name="standoff_1">
-    <visual>
-      <origin xyz="0 0 0.11"/>
-      <geometry>
-        <cylinder length="0.22" radius="0.01"/>
-      </geometry>
-      <material name="white" />
-    </visual>
-    <collision>
-      <origin xyz="0 0 0.11"/>
-      <geometry>
-        <cylinder length="0.22" radius="0.01"/>
-      </geometry>
-    </collision>
-    <inertial>
-      <mass value="0.05"/>
-      <origin xyz="0 0 0.11" rpy="0 0 0"/>
-      <inertia ixx="0.0002029" ixy="0.0" ixz="0.0" iyy="0.0002029" iyz="0.0" izz="0.0000025"/>
-    </inertial>
-  </link>
-  <joint name="joint_standoff_1" type="fixed">
-    <origin xyz="0.1 0.1 0.0775" />
-    <parent link="base_link"/>
-    <child link="standoff_1"/>
-  </joint>
+  <xacro:standoff standoff_name="standoff_1" joint_origin="0.1 0.1 0.0775" />
    <!-- Standoff 2 -->
-  <link name="standoff_2">
-    <visual>
-      <origin xyz="0 0 0.11"/>
-      <geometry>
-        <cylinder length="0.22" radius="0.01"/>
-      </geometry>
-      <material name="white" />
-    </visual>
-    <collision>
-      <origin xyz="0 0 0.11"/>
-      <geometry>
-        <cylinder length="0.22" radius="0.01"/>
-      </geometry>
-    </collision>
-    <inertial>
-      <mass value="0.05"/>
-      <origin xyz="0 0 0.11" rpy="0 0 0"/>
-      <inertia ixx="0.0002029" ixy="0.0" ixz="0.0" iyy="0.0002029" iyz="0.0" izz="0.0000025"/>
-    </inertial>
-  </link>
-  <joint name="joint_standoff_2" type="fixed">
-    <origin xyz="0.1 -0.1 0.0775" />
-    <parent link="base_link"/>
-    <child link="standoff_2"/>
-  </joint>
+  <xacro:standoff standoff_name="standoff_2" joint_origin="0.1 -0.1 0.0775" />
    <!-- Standoff 3 -->
-  <link name="standoff_3">
-    <visual>
-      <origin xyz="0 0 0.11"/>
-      <geometry>
-        <cylinder length="0.22" radius="0.01"/>
-      </geometry>
-      <material name="white" />
-    </visual>
-    <collision>
-      <origin xyz="0 0 0.11"/>
-      <geometry>
-        <cylinder length="0.22" radius="0.01"/>
-      </geometry>
-    </collision>
-    <inertial>
-      <mass value="0.05"/>
-      <origin xyz="0 0 0.11" rpy="0 0 0"/>
-      <inertia ixx="0.0002029" ixy="0.0" ixz="0.0" iyy="0.0002029" iyz="0.0" izz="0.0000025"/>
-    </inertial>
-  </link>
-  <joint name="joint_standoff_3" type="fixed">
-    <origin xyz="-0.1 -0.1 0.0775" />
-    <parent link="base_link"/>
-    <child link="standoff_3"/>
-  </joint>
+  <xacro:standoff standoff_name="standoff_3" joint_origin="-0.1 -0.1 0.0775" />
    <!-- Standoff 4 -->
-  <link name="standoff_4">
-    <visual>
-      <origin xyz="0 0 0.11"/>
-      <geometry>
-        <cylinder length="0.22" radius="0.01"/>
-      </geometry>
-      <material name="white" />
-    </visual>
-    <collision>
-      <origin xyz="0 0 0.11"/>
-      <geometry>
-        <cylinder length="0.22" radius="0.01"/>
-      </geometry>
-    </collision>
-    <inertial>
-      <mass value="0.05"/>
-      <origin xyz="0 0 0.11" rpy="0 0 0"/>
-      <inertia ixx="0.0002029" ixy="0.0" ixz="0.0" iyy="0.0002029" iyz="0.0" izz="0.0000025"/>
-    </inertial>
-  </link>
-  <joint name="joint_standoff_4" type="fixed">
-    <origin xyz="-0.1 0.1 0.0775" />
-    <parent link="base_link"/>
-    <child link="standoff_4"/>
-  </joint>
+  <xacro:standoff standoff_name="standoff_4" joint_origin="-0.1 0.1 0.0775" />
   <!-- Tray -->
-  <link name="tray">
-    <visual>
-      <origin xyz="0 0 0.045"/>
-      <geometry>
-        <cylinder length="0.09" radius="0.16"/>
-      </geometry>
-      <material name="blue" />
-    </visual>
-    <collision>
-      <origin xyz="0 0 0.045"/>
-      <geometry>
-        <cylinder length="0.09" radius="0.16"/>
-      </geometry>
-    </collision>
-    <inertial>
-      <origin xyz="0 0 0.045"/>
-      <mass value="0.3"/>
-      <inertia ixx="0.0021225" ixy="0.0" ixz="0.0" iyy="0.0021225" iyz="0.0" izz="0.00384"/>
-    </inertial>
-  </link>
-  <joint name="joint_tray" type="fixed">
-    <origin xyz="0 0 0.2975"/>
-    <parent link="base_link"/>
-    <child link="tray"/>
-  </joint>
+  <xacro:cupholder cupholder_name="tray" joint_origin="0 0 0.2975" />
   <!-- Laser Scan -->
   <link name="laser_scan_link">

Commit message: Add laser scan xacro file

File: xacro/barista_robot_model.urdf.xacro (robot description, xacro)
@@ -1,8 +1,10 @@
 <?xml version="1.0"?>
 <robot xmlns:xacro="http://www.ros.org/wiki/xacro" name="barista_robot">
+  <xacro:arg name="include_laser" default="true"/>
   <xacro:include filename="$(find barista_robot_description)/xacro/drive_wheel.xacro" />
   <xacro:include filename="$(find barista_robot_description)/xacro/caster_wheel.xacro" />
   <xacro:include filename="$(find barista_robot_description)/xacro/standoff_rod.xacro" />
   <xacro:include filename="$(find barista_robot_description)/xacro/cup_holder_tray.xacro" />
+  <xacro:include filename="$(find barista_robot_description)/xacro/laser_scanner.xacro" />
   <gazebo reference="base_link">
     <material>Gazebo/Blue</material>
@@ -119,34 +121,8 @@
   <xacro:cupholder cupholder_name="tray" joint_origin="0 0 0.2975" />
   <!-- Laser Scan -->
-  <link name="laser_scan_link">
-    <visual>
-      <origin rpy="0 0 0" xyz="0 0 0"/>
-      <geometry>
-        <mesh filename="package://barista_robot_description/meshes/hokuyo_urg_04lx.dae" scale="1.0 1.0 1.0"/>
-      </geometry>
-    </visual>
-    <collision>
-       <origin rpy="0 0 0" xyz="0 0 0.204"/>
-      <geometry>
-        <cylinder length="0.0408" radius="0.037493"/>
-      </geometry>
-    </collision>
-    <inertial>
-      <mass value="0.01"/>
-      <origin rpy="0 0 0" xyz="0 0 0.204"/>
-      <inertia ixx="6.066578520833334e-06" ixy="0" ixz="0" iyy="6.072950163333333e-06" iyz="0" izz="9.365128684166666e-06"/>
-    </inertial>
-  </link>
-  <joint name="laser_scan_link_joint" type="fixed">
-    <origin rpy="0 0 0" xyz="0.12 0 0.0775"/>
-    <parent link="base_link"/>
-    <child link="laser_scan_link"/>
-  </joint>
-  <link name="laser_scan_frame" />
-  <joint name="laser_scan_frame_joint" type="fixed">
-    <origin rpy="0 0 0" xyz="0.03 0 0.05"/>
-    <parent link="laser_scan_link"/>
-    <child link="laser_scan_frame"/>
-  </joint>
+  <xacro:if value="$(arg include_laser)">
+    <xacro:laser laser_name="laser_scan" joint_origin="0.12 0 0.0775" />
+  </xacro:if>
+  <!-- </xacro:if> -->
   <!-- Plugins -->
   <!-- Joint State Publisher -->
@@ -187,34 +163,3 @@
     </plugin>
   </gazebo>
-  <!-- Laser Scan -->
-  <gazebo reference="laser_scan_frame">
-    <sensor name="sensor_ray" type="ray">
-      <pose>0 0 0 0 0 0</pose>
-      <ray>
-        <scan>
-          <horizontal>
-            <samples>200</samples>
-            <resolution>1.0</resolution>
-            <min_angle>-1.57</min_angle>
-            <max_angle>1.57</max_angle>
-          </horizontal>
-        </scan>
-        <range>
-          <min>0.1</min>
-          <max>5</max>
-        </range>
-      </ray>
-      <always_on>true</always_on>
-      <visualize>true</visualize>
-      <update_rate>30.0</update_rate>
-      <plugin name="laser" filename="libgazebo_ros_ray_sensor.so">
-        <ros>
-          <remapping>~/out:=scan</remapping>
-          <robot_base_frame>base_link</robot_base_frame>
-          <frame_name>laser_scan_frame</frame_name>
-        </ros>
-        <output_type>sensor_msgs/LaserScan</output_type>
-      </plugin>
-    </sensor>
-  </gazebo>
 </robot>

File: xacro/caster_wheel.xacro (robot description, xacro)
@@ -1,4 +1,4 @@
 <?xml version="1.0"?>
-<robot xmlns:xacro="http://www.ros.org/wiki/xacro" name="my_box_bot">
+<robot xmlns:xacro="http://www.ros.org/wiki/xacro" name="barista_robot">
   <xacro:macro name="caster" params="caster_position joint_yaw_origin">
     <link name="${caster_position}_yaw_link">

File: xacro/cup_holder_tray.xacro (robot description, xacro)
@@ -1,4 +1,4 @@
 <?xml version="1.0"?>
-<robot xmlns:xacro="http://www.ros.org/wiki/xacro" name="my_box_bot">
+<robot xmlns:xacro="http://www.ros.org/wiki/xacro" name="barista_robot">
   <xacro:macro name="cupholder" params="cupholder_name joint_origin">
     <link name="${cupholder_name}">

File: xacro/drive_wheel.xacro (robot description, xacro)
@@ -1,4 +1,4 @@
 <?xml version="1.0"?>
-<robot xmlns:xacro="http://www.ros.org/wiki/xacro" name="my_box_bot">
+<robot xmlns:xacro="http://www.ros.org/wiki/xacro" name="barista_robot">
   <xacro:macro name="wheel" params="wheel_name joint_origin">
     <link name="${wheel_name}">

File: xacro/standoff_rod.xacro (robot description, xacro)
@@ -1,4 +1,4 @@
 <?xml version="1.0"?>
-<robot xmlns:xacro="http://www.ros.org/wiki/xacro" name="my_box_bot">
+<robot xmlns:xacro="http://www.ros.org/wiki/xacro" name="barista_robot">
   <xacro:macro name="standoff" params="standoff_name joint_origin">
     <link name="${standoff_name}">

Commit message: Fix laser scan fram id and its position

File: xacro/barista_robot_model.urdf.xacro (robot description, xacro)
@@ -122,5 +122,5 @@
   <!-- Laser Scan -->
   <xacro:if value="$(arg include_laser)">
-    <xacro:laser laser_name="laser_scan" joint_origin="0.12 0 0.0775" />
+    <xacro:laser laser_name="laser_scan" joint_origin="0.13 0 0.0775" />
   </xacro:if>
   <!-- </xacro:if> -->

File: xacro/laser_scanner.xacro (robot description, xacro)
@@ -10,13 +10,13 @@
       </visual>
       <collision>
-         <origin rpy="0 0 0" xyz="0 0 0.204"/>
+         <origin rpy="0 0 0" xyz="0 0 0.035"/>
         <geometry>
-          <cylinder length="0.0408" radius="0.037493"/>
+          <cylinder length="0.07" radius="0.025"/>
         </geometry>
       </collision>
       <inertial>
-        <mass value="0.01"/>
-        <origin rpy="0 0 0" xyz="0 0 0.204"/>
-        <inertia ixx="6.066578520833334e-06" ixy="0" ixz="0" iyy="6.072950163333333e-06" iyz="0" izz="9.365128684166666e-06"/>
+        <mass value="0.015"/>
+        <origin rpy="0 0 0" xyz="0 0 0.035"/>
+        <inertia ixx="8.47e-06" ixy="0" ixz="0" iyy="8.47e-06" iyz="0" izz="8.47e-06"/>
       </inertial>
     </link>
@@ -33,10 +33,10 @@
     </link>
     <joint name="${laser_name}_frame_joint" type="fixed">
-      <origin rpy="0 0 0" xyz="0.03 0 0.05"/>
+      <origin rpy="0 0 0" xyz="0 0 0.06"/>
       <parent link="${laser_name}_link"/>
       <child link="${laser_name}_frame"/>
     </joint>
     <!-- Laser Scan -->
-    <gazebo reference="laser_scan_frame">
+    <gazebo reference="${laser_name}_frame">
       <sensor name="sensor_ray" type="ray">
         <pose>0 0 0 0 0 0</pose>
@@ -61,8 +61,7 @@
           <ros>
             <remapping>~/out:=scan</remapping>
-            <robot_base_frame>base_link</robot_base_frame>
-            <frame_name>laser_scan_frame</frame_name>
           </ros>
           <output_type>sensor_msgs/LaserScan</output_type>
+          <frame_name>${laser_name}_frame</frame_name>
         </plugin>
       </sensor>

Commit message: Add base footprint link to barista xacro model

File: xacro/barista_robot_model.urdf.xacro (robot description, xacro)
@@ -83,4 +83,6 @@
     <color rgba="1 1 1 1"/>
   </material>
+  <!-- Base footprint link -->
+  <link name="base_footprint" />
   <!-- Base Link -->
   <link name="base_link">
@@ -102,4 +104,9 @@
     </inertial>
   </link>
+   <joint name="joint_base_link" type="fixed">
+    <origin xyz="0 0 0.0975" rpy="0 0 0"/>
+    <parent link="base_footprint"/>
+    <child link="base_link"/>
+   </joint>
   <!-- Wheel Left -->
   <xacro:wheel wheel_name="left_wheel" joint_origin="0 0.15 -0.0623"/>
@@ -159,5 +166,5 @@
     <publish_odom_tf>true</publish_odom_tf>
     <odometry_frame>odom</odometry_frame>
-    <robot_base_frame>base_link</robot_base_frame>
+    <robot_base_frame>base_footprint</robot_base_frame>
     <update_rate>30</update_rate>
     </plugin>
