Commit message: Refactor to move gazebo setting from barista model to each link file

File: xacro/barista_robot_model.urdf.xacro (robot description, xacro)
@@ -9,62 +9,4 @@
   <gazebo reference="base_link">
     <material>Gazebo/Blue</material>
-  </gazebo>
-  <gazebo reference="left_wheel">
-    <kp>1000000000000000000000000000.0</kp>
-    <kd>1000000000000000000000000000.0</kd>
-    <mu1>10.0</mu1>
-    <mu2>10.0</mu2>
-    <material>Gazebo/Black</material>
-  </gazebo>
-  <gazebo reference="right_wheel">
-    <kp>1000000000000000000000000000.0</kp>
-    <kd>1000000000000000000000000000.0</kd>
-    <mu1>10.0</mu1>
-    <mu2>10.0</mu2>
-    <material>Gazebo/Black</material>
-  </gazebo>
-  <gazebo reference="front_pitch_link">
-    <kp>1000000000000000000000000000.0</kp>
-    <kd>1000000000000000000000000000.0</kd>
-    <mu1>0.5</mu1>
-    <mu2>0.5</mu2>
-    <material>Gazebo/Green</material>
-  </gazebo>
-  <gazebo reference="back_pitch_link">
-    <kp>1000000000000000000000000000.0</kp>
-    <kd>1000000000000000000000000000.0</kd>
-    <mu1>0.5</mu1>
-    <mu2>0.5</mu2>
-    <material>Gazebo/Green</material>
-  </gazebo>
-  <gazebo reference="front_yaw_link">
-    <material>Gazebo/Blue</material>
-  </gazebo>
-  <gazebo reference="front_roll_link">
-    <material>Gazebo/Red</material>
-  </gazebo>
-  <gazebo reference="back_yaw_link">
-    <material>Gazebo/Blue</material>
-  </gazebo>
-  <gazebo reference="back_roll_link">
-    <material>Gazebo/Red</material>
-  </gazebo>
-  <gazebo reference="standoff_1">
-    <material>Gazebo/White</material>
-  </gazebo>
-  <gazebo reference="standoff_2">
-    <material>Gazebo/White</material>
-  </gazebo>
-  <gazebo reference="standoff_3">
-    <material>Gazebo/White</material>
-  </gazebo>
-  <gazebo reference="standoff_4">
-    <material>Gazebo/White</material>
-  </gazebo>
-  <gazebo reference="tray">
-    <material>Gazebo/Blue</material>
-  </gazebo>
-  <gazebo reference="laser_scan_link">
-    <material>Gazebo/Gray</material>
   </gazebo>
   <material name="black">

File: xacro/caster_wheel.xacro (robot description, xacro)
@@ -2,4 +2,17 @@
 <robot xmlns:xacro="http://www.ros.org/wiki/xacro" name="barista_robot">
   <xacro:macro name="caster" params="caster_position joint_yaw_origin">
+    <gazebo reference="${caster_position}_pitch_link">
+      <kp>1000000000000000000000000000.0</kp>
+      <kd>1000000000000000000000000000.0</kd>
+      <mu1>0.5</mu1>
+      <mu2>0.5</mu2>
+      <material>Gazebo/Green</material>
+    </gazebo>
+    <gazebo reference="${caster_position}_yaw_link">
+      <material>Gazebo/Blue</material>
+    </gazebo>
+    <gazebo reference="${caster_position}_roll_link">
+      <material>Gazebo/Red</material>
+    </gazebo>
     <link name="${caster_position}_yaw_link">
     <visual>

File: xacro/cup_holder_tray.xacro (robot description, xacro)
@@ -2,4 +2,7 @@
 <robot xmlns:xacro="http://www.ros.org/wiki/xacro" name="barista_robot">
   <xacro:macro name="cupholder" params="cupholder_name joint_origin">
+    <gazebo reference="${cupholder_name}">
+      <material>Gazebo/Blue</material>
+    </gazebo>
     <link name="${cupholder_name}">
       <visual>

File: xacro/drive_wheel.xacro (robot description, xacro)
@@ -2,4 +2,11 @@
 <robot xmlns:xacro="http://www.ros.org/wiki/xacro" name="barista_robot">
   <xacro:macro name="wheel" params="wheel_name joint_origin">
+    <gazebo reference="${wheel_name}">
+      <kp>1000000000000000000000000000.0</kp>
+      <kd>1000000000000000000000000000.0</kd>
+      <mu1>10.0</mu1>
+      <mu2>10.0</mu2>
+      <material>Gazebo/Black</material>
+    </gazebo>
     <link name="${wheel_name}">
       <visual>

File: xacro/laser_scanner.xacro (robot description, xacro)
@@ -2,4 +2,7 @@
 <robot xmlns:xacro="http://www.ros.org/wiki/xacro" name="barista_robot">
   <xacro:macro name="laser" params="laser_name joint_origin">
+    <gazebo reference="${laser_name}_link">
+      <material>Gazebo/Gray</material>
+    </gazebo>
     <link name="${laser_name}_link">
       <visual>

File: xacro/standoff_rod.xacro (robot description, xacro)
@@ -2,4 +2,7 @@
 <robot xmlns:xacro="http://www.ros.org/wiki/xacro" name="barista_robot">
   <xacro:macro name="standoff" params="standoff_name joint_origin">
+     <gazebo reference="${standoff_name}">
+      <material>Gazebo/White</material>
+    </gazebo>
     <link name="${standoff_name}">
       <visual>

Commit message: Add namespace for 2 robots

File: xacro/barista_robot_model.urdf.xacro (robot description, xacro)
@@ -2,4 +2,5 @@
 <robot xmlns:xacro="http://www.ros.org/wiki/xacro" name="barista_robot">
   <xacro:arg name="include_laser" default="true"/>
+  <xacro:property name="robot_name" value="$(arg robot_name)"/>
   <xacro:include filename="$(find barista_robot_description)/xacro/drive_wheel.xacro" />
   <xacro:include filename="$(find barista_robot_description)/xacro/caster_wheel.xacro" />
@@ -71,5 +72,5 @@
   <!-- Laser Scan -->
   <xacro:if value="$(arg include_laser)">
-    <xacro:laser laser_name="laser_scan" joint_origin="0.13 0 0.0775" />
+    <xacro:laser laser_name="laser_scan" joint_origin="0.13 0 0.0775" robot_name="${robot_name}" />
   </xacro:if>
   <!-- </xacro:if> -->
@@ -79,5 +80,6 @@
     <plugin name="barista_bot_joint_state" filename="libgazebo_ros_joint_state_publisher.so">
     <ros>
-        <remapping>~/out:=joint_states</remapping>
+      <namespace>/${robot_name}</namespace>
+      <remapping>~/out:=joint_states</remapping>
     </ros>
     <update_rate>30</update_rate>
@@ -95,4 +97,8 @@
   <gazebo>
     <plugin filename="libgazebo_ros_diff_drive.so" name="differential_drive_controller">
+    <ros>
+      <namespace>/${robot_name}</namespace>
+      <remapping>/cmd_vel:=cmd_vel</remapping>
+    </ros>
     <!-- wheels -->
     <left_joint>joint_left_wheel</left_joint>
@@ -107,6 +113,6 @@
     <publish_odom>true</publish_odom>
     <publish_odom_tf>true</publish_odom_tf>
-    <odometry_frame>odom</odometry_frame>
-    <robot_base_frame>base_footprint</robot_base_frame>
+    <odometry_frame>${robot_name}/odom</odometry_frame>
+    <robot_base_frame>${robot_name}/base_footprint</robot_base_frame>
     <update_rate>30</update_rate>
     </plugin>

File: xacro/laser_scanner.xacro (robot description, xacro)
@@ -1,5 +1,5 @@
 <?xml version="1.0"?>
 <robot xmlns:xacro="http://www.ros.org/wiki/xacro" name="barista_robot">
-  <xacro:macro name="laser" params="laser_name joint_origin">
+  <xacro:macro name="laser" params="laser_name joint_origin robot_name">
     <gazebo reference="${laser_name}_link">
       <material>Gazebo/Gray</material>
@@ -63,4 +63,5 @@
         <plugin name="laser" filename="libgazebo_ros_ray_sensor.so">
           <ros>
+            <namespace>/${robot_name}</namespace>
             <remapping>~/out:=scan</remapping>
           </ros>

Commit message: Add color to barista robot based on its name

File: xacro/barista_robot_model.urdf.xacro (robot description, xacro)
@@ -9,5 +9,10 @@
   <xacro:include filename="$(find barista_robot_description)/xacro/laser_scanner.xacro" />
   <gazebo reference="base_link">
-    <material>Gazebo/Blue</material>
+    <xacro:if value="${robot_name == 'morty'}">
+      <material>Gazebo/Blue</material>
+    </xacro:if>
+    <xacro:if value="${robot_name == 'rick'}">
+      <material>Gazebo/Red</material>
+    </xacro:if>
   </gazebo>
   <material name="black">
@@ -34,5 +39,10 @@
         <cylinder length="0.155" radius="0.178" />
       </geometry>
-      <material name="blue" />
+      <xacro:if value="${robot_name == 'morty'}">
+        <material name="blue" />
+      </xacro:if>
+      <xacro:if value="${robot_name == 'rick'}">
+        <material name="red" />
+      </xacro:if>
     </visual>
     <collision>
@@ -69,5 +79,5 @@
   <xacro:standoff standoff_name="standoff_4" joint_origin="-0.1 0.1 0.0775" />
   <!-- Tray -->
-  <xacro:cupholder cupholder_name="tray" joint_origin="0 0 0.2975" />
+  <xacro:cupholder cupholder_name="tray" joint_origin="0 0 0.2975" robot_name="${robot_name}"/>
   <!-- Laser Scan -->
   <xacro:if value="$(arg include_laser)">

File: xacro/cup_holder_tray.xacro (robot description, xacro)
@@ -1,7 +1,12 @@
 <?xml version="1.0"?>
 <robot xmlns:xacro="http://www.ros.org/wiki/xacro" name="barista_robot">
-  <xacro:macro name="cupholder" params="cupholder_name joint_origin">
+  <xacro:macro name="cupholder" params="cupholder_name joint_origin robot_name">
     <gazebo reference="${cupholder_name}">
-      <material>Gazebo/Blue</material>
+      <xacro:if value="${robot_name == 'morty'}">
+        <material>Gazebo/Blue</material>
+      </xacro:if>
+      <xacro:if value="${robot_name == 'rick'}">
+        <material>Gazebo/Red</material>
+      </xacro:if>
     </gazebo>
     <link name="${cupholder_name}">
@@ -11,5 +16,10 @@
           <cylinder length="0.09" radius="0.16"/>
         </geometry>
-        <material name="blue" />
+        <xacro:if value="${robot_name == 'morty'}">
+          <material name="blue" />
+        </xacro:if>
+        <xacro:if value="${robot_name == 'rick'}">
+          <material name="red" />
+        </xacro:if>
       </visual>
       <collision>
